File: PCB/Advik's Hackpad.kicad_pcb (KiCad board)
At the start: 2 copper layers, 62 x 64 mm, 8 parts, among them SW1 SW_Push, SW2 SW_Push, SW3 SW_Push, SW4 SW_Push, SW5 SW_Push, U1 XIAO-RP2040-DIP

Commit message: Add files via upload
Parts:
- removed C1: C, Capacitor_SMD:C_0805_2012Metric
Routing:
- net +5V: track 40.8 -> 30.3 mm
- net Net-(D1-DIN): track 57.3 -> 58.9 mm
- net GND: track 130.7 -> 130.1 mm
Other:
- board text added: "Advik's KEYPAD v3.4.2 (F) by ADVANCED START"
- board text removed: "Advik's KEYPAD v3.4.0 (F) by ADVANCED START"
Changed lines of the file:
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@@
 			(at 0 -2.75 0)
 			(layer "F.SilkS")
+			(hide yes)
 			(effects
 				(font
@@
 			(fill no)
 			(layer "F.Fab")
-		)
-		(fp_text user "1"
-			(at -3.71 -1.005 0)
-			(unlocked yes)
-			(layer "F.SilkS")
-			(effects
-				(font
-					(size 0.8 0.8)
-					(thickness 0.15)
-				)
-			)
 		)
 		(fp_text user "${REFERENCE}"
@@
 		)
 	)
-	(footprint "Capacitor_SMD:C_0805_2012Metric"
-		(layer "F.Cu")
-		(at 167.859 78.914 90)
-		(descr "Capacitor SMD 0805 (2012 Metric), square (rectangular) end terminal, IPC-7351 nominal, (Body size source: IPC-SM-782 page 76, https://www.pcb-3d.com/wordpress/wp-content/uploads/ipc-sm-782a_amendment_1_and_2.pdf, https://docs.google.com/spreadsheets/d/1BsfQQcO9C6DZCsRaXUlFlo91Tg2WpOkGARC1WS5S8t0/edit?usp=sharing), generated with kicad-footprint-generator")
-		(tags "capacitor")
-		(property "Reference" "C1"
-			(at 0 -1.68 90)
-			(layer "F.SilkS")
-			(hide yes)
-			(effects
-				(font
-					(size 1 1)
-					(thickness 0.15)
-				)
-			)
-		)
-		(property "Value" "C"
-			(at 0 1.68 90)
-			(layer "F.Fab")
-			(effects
-				(font
-					(size 1 1)
-					(thickness 0.15)
-				)
-			)
-		)
-		(property "Datasheet" "~"
-			(at 0 0 90)
-			(layer "F.Fab")
-			(hide yes)
-			(effects
-				(font
-					(size 1.27 1.27)
-					(thickness 0.15)
-				)
-			)
-		)
-		(property "Description" "Unpolarized capacitor"
-			(at 0 0 90)
-			(layer "F.Fab")
-			(hide yes)
-			(effects
-				(font
-					(size 1.27 1.27)
-					(thickness 0.15)
-				)
-			)
-		)
-		(property ki_fp_filters "C_*")
-		(sheetname "/")
-		(sheetfile "Advik's Hackpad.kicad_sch")
-		(attr smd)
-		(fp_line
-			(start -0.261252 -0.735)
-			(end 0.261252 -0.735)
-			(stroke
-				(width 0.12)
-				(type solid)
-			)
-			(layer "F.SilkS")
-		)
-		(fp_line
-			(start -0.261252 0.735)
-			(end 0.261252 0.735)
-			(stroke
-				(width 0.12)
-				(type solid)
-			)
-			(layer "F.SilkS")
-		)
-		(fp_rect
-			(start -1.7 -0.98)
-			(end 1.7 0.98)
-			(stroke
-				(width 0.05)
-				(type solid)
-			)
-			(fill no)
-			(layer "F.CrtYd")
-		)
-		(fp_rect
-			(start -1 -0.625)
-			(end 1 0.625)
-			(stroke
-				(width 0.1)
-				(type solid)
-			)
-			(fill no)
-			(layer "F.Fab")
-		)
-		(fp_text user "${REFERENCE}"
-			(at 0 0 90)
-			(layer "F.Fab")
-			(effects
-				(font
-					(size 0.5 0.5)
-					(thickness 0.08)
-				)
-			)
-		)
-		(pad "1" smd roundrect
-			(at -0.95 0 90)
-			(size 1 1.45)
-			(layers "F.Cu" "F.Mask" "F.Paste")
-			(roundrect_rratio 0.25)
-			(net 2 "+5V")
-			(pintype "passive")
-		)
-		(pad "2" smd roundrect
-			(at 0.95 0 90)
-			(size 1 1.45)
-			(layers "F.Cu" "F.Mask" "F.Paste")
-			(roundrect_rratio 0.25)
-			(net 1 "GND")
-			(pintype "passive")
-		)
-		(embedded_fonts no)
-		(model "${KICAD9_3DMODEL_DIR}/Capacitor_SMD.3dshapes/C_0805_2012Metric.step"
-			(offset
-				(xyz 0 0 0)
-			)
-			(scale
-				(xyz 1 1 1)
-			)
-			(rotate
-				(xyz 0 0 0)
-			)
-		)
-	)
 	(footprint "Button_Switch_Keyboard:SW_Cherry_MX_1.00u_PCB"
 		(layer "F.Cu")
@@
 		)
 	)
-	(gr_text "Advik's \nKEYPAD\nv3.4.0 (F)\nby ADVANCED START"
+	(gr_text "Advik's \nKEYPAD\nv3.4.2 (F)\nby ADVANCED START"
 		(at 121.05 64.18 0)
 		(layer "F.SilkS")
@@
 	)
 	(segment
-		(start 163.155 82.668)
-		(end 167.859 77.964)
+		(start 163.155 102.71)
+		(end 163.155 86.218)
 		(width 0.2)
 		(layer "F.Cu")
@@
 	)
 	(segment
-		(start 167.859 77.964)
-		(end 167.859 71.224)
+		(start 171.299 78.074)
+		(end 171.299 74.664)
 		(width 0.2)
 		(layer "F.Cu")
@@
 	)
 	(segment
-		(start 167.859 71.224)
+		(start 171.299 74.664)
 		(end 156.335 59.7)
 		(width 0.2)
@@
 	)
 	(segment
-		(start 168.349 78.074)
-		(end 171.299 78.074)
-		(width 0.2)
-		(layer "F.Cu")
-		(net 1)
-	)
-	(segment
-		(start 167.859 77.964)
-		(end 168.239 77.964)
-		(width 0.2)
-		(layer "F.Cu")
-		(net 1)
-	)
-	(segment
 		(start 125.1 83.66)
 		(end 144.15 83.66)
@@
 	)
 	(segment
-		(start 163.155 102.71)
-		(end 163.155 82.668)
-		(width 0.2)
-		(layer "F.Cu")
-		(net 1)
-	)
-	(segment
 		(start 144.15 102.71)
 		(end 163.2 102.71)
@@
 	)
 	(segment
+		(start 163.155 86.218)
+		(end 171.299 78.074)
+		(width 0.2)
+		(layer "F.Cu")
+		(net 1)
+	)
+	(segment
 		(start 156.57763 59.7)
 		(end 155.5 59.7)
@@
 	)
 	(segment
-		(start 168.239 77.964)
-		(end 168.349 78.074)
-		(width 0.2)
-		(layer "F.Cu")
-		(net 1)
-	)
-	(segment
 		(start 163.38625 102.71)
 		(end 163.41125 102.735)
@@
 	)
 	(segment
-		(start 168.875 80.55)
-		(end 174.073 80.55)
+		(start 174.799 79.824)
+		(end 173.6 78.625)
 		(width 0.2)
 		(layer "F.Cu")
@@
 	)
 	(segment
-		(start 174.073 80.55)
-		(end 174.799 79.824)
+		(start 173.6 78.625)
+		(end 173.6 74.425)
 		(width 0.2)
 		(layer "F.Cu")
@@
 	)
 	(segment
-		(start 168.923 78.8)
-		(end 172.4 78.8)
+		(start 173.6 74.425)
+		(end 156.335 57.16)
 		(width 0.2)
 		(layer "F.Cu")
@@
 	)
 	(segment
-		(start 167.859 79.864)
-		(end 168.539 80.544)
-		(width 0.2)
-		(layer "F.Cu")
-		(net 2)
-	)
-	(segment
-		(start 172.4 73.225)
-		(end 156.335 57.16)
-		(width 0.2)
-		(layer "F.Cu")
-		(net 2)
-	)
-	(segment
-		(start 172.4 78.8)
-		(end 172.4 73.225)
-		(width 0.2)
-		(layer "F.Cu")
-		(net 2)
-	)
-	(segment
-		(start 167.859 79.864)
-		(end 168.923 78.8)
-		(width 0.2)
-		(layer "F.Cu")
-		(net 2)
-	)
-	(segment
-		(start 168.869 80.544)
-		(end 168.875 80.55)
-		(width 0.2)
-		(layer "F.Cu")
-		(net 2)
-	)
-	(segment
-		(start 168.539 80.544)
-		(end 168.869 80.544)
-		(width 0.2)
-		(layer "F.Cu")
-		(net 2)
-	)
-	(segment
-		(start 175.9 78.8)
+		(start 151.483 56.097)
+		(end 140.26 67.32)
+		(width 0.2)
+		(layer "F.Cu")
+		(net 4)
+	)
+	(segment
+		(start 157.590626 56.097)
+		(end 151.483 56.097)
+		(width 0.2)
+		(layer "F.Cu")
+		(net 4)
+	)
+	(segment
+		(start 175.9 80.55)
 		(end 175.9 74.406374)
 		(width 0.2)
@@
 	(segment
 		(start 171.299 79.824)
-		(end 172.674 79.824)
-		(width 0.2)
-		(layer "F.Cu")
-		(net 4)
-	)
-	(segment
-		(start 172.674 79.824)
-		(end 173.698 78.8)
-		(width 0.2)
-		(layer "F.Cu")
-		(net 4)
-	)
-	(segment
-		(start 173.698 78.8)
-		(end 175.9 78.8)
+		(end 172.025 80.55)
 		(width 0.2)
 		(layer "F.Cu")
@@
 	)
 	(segment
-		(start 157.590626 56.097)
-		(end 151.483 56.097)
-		(width 0.2)
-		(layer "F.Cu")
-		(net 4)
-	)
-	(segment
-		(start 151.483 56.097)
-		(end 140.26 67.32)
+		(start 172.025 80.55)
+		(end 175.9 80.55)
 		(width 0.2)
 		(layer "F.Cu")
@@
 	)
 	(segment
+		(start 169.505 100.17)
+		(end 169.505 81.325)
+		(width 0.2)
+		(layer "B.Cu")
+		(net 9)
+	)
+	(segment
 		(start 169.505 81.325)
 		(end 155.5 67.32)
 		(width 0.2)
 		(layer "B.Cu")
-		(net 9)
-	)
-	(segment
-		(start 169.505 100.17)
-		(end 169.505 81.325)
-		(width 0.2)
-		(layer "B.Cu")
